File: gps-radio-beacon.kicad_sch (KiCad schematic)
At the start: 40 parts, among them J1 Conn_01x02, J2 Conn_Coaxial, J3 Conn_Coaxial, SW1 SW_Push, U1 RP2040, U2 MAX-M10S, U3 W25Q128JVS, Y1 Crystal

Commit message: redesign pim
Parts:
- removed C10, C11, C14, C15, C16, C18, C4, C5, C7, C9: 100n, Capacitor_THT:CP_Radial_Tantal_D4.5mm_P2.50mm, symbol Device:C
- removed C12, C13: 27p, symbol Device:C
- removed C3, C6, C8: 1u, Capacitor_THT:CP_Radial_Tantal_D4.5mm_P2.50mm, symbol Device:C
- removed D1: LED, symbol Device:LED
- removed J1: Conn_01x02, symbol Connector_Generic:Conn_01x02
- removed R3: 200, symbol Device:R
- removed R4, R5, R6: 4.7k, symbol Device:R
- removed R7: 1k, symbol Device:R
- removed SW1: SW_Push, symbol Switch:SW_Push
- removed U1: RP2040, Package_DFN_QFN:QFN-56-1EP_7x7mm_P0.4mm_EP3.2x3.2mm, symbol MCU_RaspberryPi:RP2040
- removed U3: W25Q128JVS, Package_SO:SOIC-8_5.23x5.23mm_P1.27mm, symbol Memory_Flash:W25Q128JVS
- removed Y1: Crystal, symbol Device:Crystal
- added U1: PGA2040, grb:PGA2040, symbol grb:PGA2040
- added U2: Si4463, Package_DFN_QFN:QFN-20-1EP_4x4mm_P0.5mm_EP2.6x2.6mm_ThermalVias, symbol RF:Si4463
- C2: value 100n -> 4.7n; footprint Capacitor_THT:CP_Radial_Tantal_D4.5mm_P2.50mm -> Capacitor_SMD:C_1206_3216Metric_Pad1.33x1.80mm_HandSolder
- C3: renamed from C17; footprint (none) -> Capacitor_SMD:C_1206_3216Metric_Pad1.33x1.80mm_HandSolder
- H1, H2, H3, H4: footprint (none) -> MountingHole:MountingHole_3.2mm_M3
- J3: renamed from J2; footprint (none) -> Connector_Coaxial:SMA_Molex_73251-1153_EdgeMount_Horizontal
- J4: renamed from J3; footprint (none) -> Connector_Coaxial:SMA_Molex_73251-1153_EdgeMount_Horizontal
- L1: footprint (none) -> Inductor_SMD:L_0402_1005Metric
- R1, R2: value 27.4 -> 4.7k; footprint (none) -> Resistor_THT:R_Axial_DIN0207_L6.3mm_D2.5mm_P10.16mm_Horizontal
- TP1: footprint (none) -> TestPoint:TestPoint_Loop_D2.54mm_Drill1.5mm_Beaded
- renumbered U2 to U3
Connections:
- net +3V3: now also U1.B3 (3V3), U2.6 (VDD), U2.8 (VDD)
- net AFSK_SIGNAL: now also C2.1, R2.2, U2.17 (XIN); no longer J3.1 (In)
- net GND: now also R1.2, U1.A1 (GND), U1.A3 (3V3_EN), U1.A8, U1.B2, U1.B7, U1.G2, U1.G7, U1.H1, U1.H8, U2.1 (SDN), U2.18 (GND), U2.21 (GND); no longer C1.2
- net GPS_SCL: now also U1.C8 (GPIO27)
- net GPS_SDA: now also U1.D7 (GPIO26)
- net PWR-USB/USB_D+: now also U1.A5 (USB_DP); no longer R1.1
- net PWR-USB/USB_D-: now also U1.A6 (USB_DM); no longer R2.1
- net +1V1: no longer names the net of C1.1
- net +1V1: now also U1.B1 (GPIO0); no longer C2.1
- new net: C1.2, R1.1, R2.1
- new net: J3.1 (In), U2.4 (TX)
- new net RADIO_MISO: U1.G8 (GPIO20), U2.13 (SDO)
- new net RADIO_MOSI: U1.H7 (GPIO19), U2.14 (SDI)
- new net RADIO_SCLK: U1.G6 (GPIO18), U2.12 (SCLK)
- new net ~{RADIO_CS}: U1.F8 (GPIO21), U2.15 (~{SEL})
- new net ~{RADIO_INT}: U1.E8 (GPIO23), U2.11 (~{IRQ})
- no-connect marks 31 -> 43
Other:
- note added: "@Adian: This is a band pass filter."
- note added: "High pass filter"
- note added: "Low pass filter"
- note removed: "According to _Hardware Design with the RP2040_, we do not need a pull up resistor here."
- note removed: "I think we need to put an actual radio in between here, but I'm waiting on Zack's CDR to pick one first. Right now, this should work for listening, but not transmitting."
- note removed: "Reset"
- note removed: "These SPI wires shoud be short for data integrity."
- note removed: "These resistors should be placed close to RP2040 pins 46 and 47"
- note removed: "This capacitor should be placed close to RP2040 pin 10"
- note removed: "This capacitor should be placed close to RP2040 pin 45"
- moved on the sheet: C3, J3, J4, L1, U3

Commit message: redesign for use with RFM95
Parts:
- removed C1: 100n, Capacitor_THT:CP_Radial_Tantal_D4.5mm_P2.50mm, symbol Device:C
- removed C2: 4.7n, Capacitor_SMD:C_1206_3216Metric_Pad1.33x1.80mm_HandSolder, symbol Device:C
- removed R1, R2: 4.7k, Resistor_THT:R_Axial_DIN0207_L6.3mm_D2.5mm_P10.16mm_Horizontal, symbol Device:R
- removed TP1: TestPoint, TestPoint:TestPoint_Loop_D2.54mm_Drill1.5mm_Beaded, symbol Connector:TestPoint
- removed U2: Si4463, Package_DFN_QFN:QFN-20-1EP_4x4mm_P0.5mm_EP2.6x2.6mm_ThermalVias, symbol RF:Si4463
- added C4: 10u, Capacitor_SMD:C_1206_3216Metric_Pad1.33x1.80mm_HandSolder, symbol Device:C
- added D3: LED, LED_THT:LED_D3.0mm, symbol Device:LED
- added J5: Screw_Terminal_01x04, TerminalBlock_Phoenix:TerminalBlock_Phoenix_MKDS-1,5-4-5.08_1x04_P5.08mm_Horizontal, symbol Connector:Screw_Terminal_01x04
- added R3, R8: 200, Resistor_SMD:R_0805_2012Metric_Pad1.20x1.40mm_HandSolder, symbol Device:R
- added R4, R7: 10k, Resistor_SMD:R_0805_2012Metric_Pad1.20x1.40mm_HandSolder, symbol Device:R
- added U2: RFM95W-915S2, RF_Module:HOPERF_RFM9XW_SMD, symbol RF_Module:RFM95W-915S2
- L1: footprint Inductor_SMD:L_0402_1005Metric -> Inductor_SMD:L_1210_3225Metric_Pad1.42x2.65mm_HandSolder
- renumbered C3 to C1
Connections:
- net +3V3: now also C4.2, R4.1, R7.1, U2.13 (3.3V)
- net GND: now also C4.1, R3.2, R8.2, U2.1 (GND), U2.10 (GND), U2.8 (GND)
- net GPS_TIMEPULSE: now also U1.H3 (GPIO11)
- net RADIO_MISO: now also U1.D2 (GPIO4), U2.2 (MISO); no longer U1.G8 (GPIO20)
- net RADIO_MOSI: now also U1.F1 (GPIO7), U2.3 (MOSI); no longer U1.H7 (GPIO19)
- net at J3.1 (In): now also U2.9 (ANT)
- net at U1.D8 (GPIO25): now also D3.2 (A)
- net RADIO_CS: now reaches U1.E1 (GPIO5)
- net RADIO_CS: now also U2.5 (NSS)
- net RADIO_SCK: now reaches U1.E2 (GPIO6)
- net RADIO_SCK: now also U2.4 (SCK)
- net RADIO_IRQ: now reaches U1.F2 (GPIO8)
- net RADIO_IRQ: now also U2.14 (DIO0)
- net RADIO_RESET: now reaches U1.G1 (GPIO9)
- net RADIO_RESET: now also R4.2, U2.6 (RESET)
- net IND_LED_2: now reaches U1.G4 (GPIO14)
- net IND_LED_2: now also J5.3 (Pin_3)
- net GPS_RESET: now reaches U1.H2 (GPIO10)
- net GPS_RESET: now also U3.9 (~{RESET}), R7.2
- net IND_LED_1: now reaches U1.H4 (GPIO13)
- net IND_LED_1: now also J5.2 (Pin_2)
- net IND_LED_3: now reaches U1.H5 (GPIO15)
- net IND_LED_3: now also J5.4 (Pin_4)
- net RADIO_SCLK: no longer names the net of U1.G6 (GPIO18)
- net ~{RADIO_CS}: no longer names the net of U1.F8 (GPIO21)
- net ~{RADIO_INT}: no longer names the net of U1.E8 (GPIO23)
- new net: J5.1 (Pin_1), R8.1
- new net: D3.1 (K), R3.1
- no-connect marks 43 -> 33
Other:
- note added: "GPS"
- note added: "Indicator LED"
- note added: "Microcontroller"
- note added: "Radio Module"
- note removed: "@Adian: This is a band pass filter."
- note removed: "High pass filter"
- note removed: "Low pass filter"
- note removed: "This little circuit is a bias tee, it's reccomended for use with the GPS."
- moved on the sheet: C1, J4, L1, U1, U3

Commit message: Add BOOTSEL button
Parts:
- added SW1: SW_Push, Button_Switch_THT:SW_PUSH_6mm, symbol Switch:SW_Push
Connections:
- net GND: now also SW1.1
- net at U1.A7 (BOOTSEL): now also SW1.2
- no-connect marks 33 -> 32

Commit message: Fix many bugs with the initial version
Parts:
- removed C1: 10n, Capacitor_SMD:C_1206_3216Metric_Pad1.33x1.80mm_HandSolder, symbol Device:C
- removed J4: Conn_Coaxial, Connector_Coaxial:SMA_Molex_73251-1153_EdgeMount_Horizontal, symbol Connector:Conn_Coaxial
- removed L1: 27n, Inductor_SMD:L_1210_3225Metric_Pad1.42x2.65mm_HandSolder, symbol Device:L
- removed U3: MAX-M10S, RF_GPS:ublox_MAX, symbol GRB-HW:MAX-M10S
- added U3: Adafruit_Ultimate_GPS_Breakout, grb:Adafruit_Ultimate_GPS_Breakout, symbol grb:Adafruit_Ultimate_GPS_Breakout
Connections:
- net +3V3: now also U3.8 (VIN)
- net GND: now also U3.7 (GND)
- net RADIO_RESET: now also U1.D1 (GPIO3); no longer U1.G1 (GPIO9)
- net RADIO_DIO3: now reaches U2.11 (DIO3)
- net RADIO_DIO3: now also U1.G6 (GPIO18)
- net RADIO_DIO4: now reaches U2.12 (DIO4)
- net RADIO_DIO4: now also U1.H6 (GPIO17)
- net RADIO_DIO1: now reaches U2.15 (DIO1)
- net RADIO_DIO1: now also U1.G8 (GPIO20)
- net RADIO_DIO2: now reaches U2.16 (DIO2)
- net RADIO_DIO2: now also U1.H7 (GPIO19)
- net RADIO_DIO5: now reaches U2.7 (DIO5)
- net RADIO_DIO5: now also U1.G5 (GPIO16)
- net VBUS: now reaches U1.A2 (VBUS)
- net RADIO_DIO0: now reaches U1.F8 (GPIO21)
- net RADIO_DIO0: now also U2.14 (DIO0)
- net GPS_RESET renamed GPS_EN
- net GPS_EN: now also U1.F2 (GPIO8), U3.2 (EN); no longer U1.H2 (GPIO10)
- net GPS_SCL: no longer names the net of U1.C8 (GPIO27)
- net GPS_SDA: no longer names the net of U1.D7 (GPIO26)
- net GPS_TIMEPULSE: no longer names the net of U1.H3 (GPIO11)
- removed net RADIO_IRQ: U1.F2 (GPIO8), U2.14 (DIO0)
- new net GPS_RX: U1.H2 (GPIO10), U3.6 (RX)
- new net GPS_TX: U1.G1 (GPIO9), U3.5 (TX)
- no-connect marks 32 -> 20
Other:
- moved on the sheet: C4, D3, J3, R3, R4, U2

Commit message: Final changes for comp
Parts:
- removed J5: Screw_Terminal_01x04, TerminalBlock_Phoenix:TerminalBlock_Phoenix_MKDS-1,5-4-5.08_1x04_P5.08mm_Horizontal, symbol Connector:Screw_Terminal_01x04
- removed R7: 10k, Resistor_SMD:R_0805_2012Metric_Pad1.20x1.40mm_HandSolder, symbol Device:R
- removed SW1: SW_Push, Button_Switch_THT:SW_PUSH_6mm, symbol Switch:SW_Push
- removed U1: PGA2040, grb:PGA2040, symbol grb:PGA2040
- added D2: 1N5228BTR, Diode_THT:D_DO-35_SOD27_P7.62mm_Horizontal, symbol Device:D_Zener
- added F1: 0466.500NR, Fuse:Fuse_1206_3216Metric_Pad1.42x1.75mm_HandSolder, symbol Device:Fuse
- added J1: Conn_01x04, Connector_JST:JST_XH_S4B-XH-A_1x04_P2.50mm_Horizontal, symbol Connector_Generic:Conn_01x04
- added J3: Conn_01x02, Connector_JST:JST_XH_S2B-XH-A_1x02_P2.50mm_Horizontal, symbol Connector_Generic:Conn_01x02
- added JLong1: Conn_01x16, Connector_PinHeader_2.54mm:PinHeader_1x16_P2.54mm_Vertical, symbol Connector_Generic:Conn_01x16
- added JShort1: Conn_01x02, Connector_PinSocket_2.54mm:PinSocket_1x02_P2.54mm_Vertical, symbol Connector_Generic:Conn_01x02
- added TP1, TP10, TP11, TP12, TP13, TP14, TP15, TP16, TP17, TP18, TP19, TP2, TP20, TP3, TP4, TP5, TP6, TP7, TP8, TP9: TestPoint, TestPoint:TestPoint_Keystone_5000-5004_Miniature, symbol Connector:TestPoint
- added U1: Pico, RPi_Pico:RPi_Pico_SMD_TH, symbol RPi_Pico:Pico
- renumbered C4 to C1, D3 to D1, J3 to J2, R3 to R1, R8 to R2, R4 to R3, U3 to U2, U2 to U3
Connections:
- net +3V3: now also F1.2, U1.40 (VBUS)
- net GND: now also D2.2 (A), JLong1.2 (Pin_2), JShort1.2 (Pin_2), U1.13 (GND), U1.18 (GND), U1.23 (GND), U1.28 (GND), U1.3 (GND), U1.38 (GND), U1.42 (GND), U1.8 (GND)
- net GPS_EN: now also TP6.1, U1.11 (GPIO8)
- net GPS_RX: now also TP8.1, U1.14 (GPIO10)
- net GPS_TX: now also TP7.1, U1.12 (GPIO9)
- net IND_LED_1: now also J1.2 (Pin_2), J3.2 (Pin_2), TP9.1, U1.17 (GPIO13)
- net IND_LED_2: now also J1.3 (Pin_3), TP10.1, U1.19 (GPIO14)
- net IND_LED_3: now also J1.4 (Pin_4), TP11.1, U1.20 (GPIO15)
- net RADIO_CS: now also TP3.1, U1.7 (GPIO5)
- net RADIO_DIO0: now also TP12.1, U1.27 (GPIO21)
- net RADIO_DIO1: now also TP13.1, U1.26 (GPIO20)
- net RADIO_DIO2: now also TP14.1, U1.25 (GPIO19)
- net RADIO_DIO3: now also TP15.1, U1.24 (GPIO18)
- net RADIO_DIO4: now also TP16.1, U1.22 (GPIO17)
- net RADIO_DIO5: now also TP17.1, U1.21 (GPIO16)
- net RADIO_MISO: now also TP2.1, U1.6 (GPIO4)
- net RADIO_MOSI: now also TP5.1, U1.10 (GPIO7)
- net RADIO_RESET: now also TP1.1, U1.5 (GPIO3)
- net RADIO_SCK: now also TP4.1, U1.9 (GPIO6)
- net at R2.1: now also J1.1 (Pin_1), J3.1 (Pin_1)
- net at U2.1 (3V3): now also TP18.1
- net at U2.4 (FIX): now also TP19.1
- net at U2.9 (PPS): now also TP20.1
- net at D1.2 (A): now also U1.31 (GPIO26_ADC0)
- new net VCC: D2.1 (K), F1.1, JLong1.1 (Pin_1), JShort1.1 (Pin_1)
- no-connect marks 20 -> 31
Other:
- removed sheet PWR-USB
- note added: "Circuit Protection"
- note added: "Header Pins"
- note added: "Indicator LEDs"
- note removed: "Indicator LED"
- moved on the sheet: C1, D1, J2, R1, R2, R3, U2, U3
